Commit message: change package naming, remove unnecesary files

File: urdf/model.urdf.xacro (robot description, xacro)
@@ -1,5 +1,5 @@
 <?xml version="1.0" encoding="UTF-8"?>
 <robot xmlns:xacro="http://www.ros.org/wiki/xacro" name="rover">
-    <xacro:include filename="$(find nano)/urdf/wheel.xacro" />
+    <xacro:include filename="$(find aio_robot)/urdf/wheel.xacro" />
     <link name="base_footprint" pose="0 0 0 0 0 0" />
     <link name="base_link">
@@ -47,5 +47,5 @@
             <origin xyz="0 0 0" rpy="0 0 0" />
             <geometry>
-                <mesh filename="package://nano/meshes/hokuyo.dae" />
+                <mesh filename="package://aio_robot/meshes/hokuyo.dae" />
             </geometry>
         </visual>
@@ -58,5 +58,5 @@
     <joint name="hokuyo_joint" type="fixed">
         <axis xyz="0 1 0" />
-        <origin xyz="0.0 0.00 0.06" rpy="0 0 0" /><!--"0 0 1.5707 for andrew case"-->
+        <origin xyz="0.0 0.00 0.06" rpy="0 0 0" />
         <parent link="base_link" />
         <child link="laser" />

File: urdf/model_sim.urdf.xacro (robot description, xacro)
@@ -1,6 +1,6 @@
 <?xml version="1.0" encoding="UTF-8"?>
 <robot xmlns:xacro="http://www.ros.org/wiki/xacro" name="rover">
-    <xacro:include filename="$(find nano)/urdf/wheel.xacro" />
-    <xacro:include filename="$(find nano)/urdf/gaz.xacro" />
+    <xacro:include filename="$(find aio_robot)/urdf/wheel.xacro" />
+    <xacro:include filename="$(find aio_robot)/urdf/gaz.xacro" />
     <link name="base_footprint" pose="0 0 0 0 0 0" />
     <link name="base_link">
@@ -48,5 +48,5 @@
             <origin xyz="0 0 0" rpy="0 0 0" />
             <geometry>
-                <mesh filename="package://nano/meshes/hokuyo.dae" />
+                <mesh filename="package://aio_robot/meshes/hokuyo.dae" />
             </geometry>
         </visual>

File: urdf/wheel.xacro (robot description, xacro)
@@ -6,5 +6,5 @@
                 <geometry>
                     <!--cylinder length=".1" radius="0.13" /-->
-                    <mesh filename="package://nano/meshes/wheel.dae" scale="0.6 0.6 0.6" />
+                    <mesh filename="package://aio_robot/meshes/wheel.dae" scale="0.6 0.6 0.6" />
                 </geometry>
                 <origin rpy="${rot} 0 0" xyz="0 0 0.0" />
@@ -13,5 +13,5 @@
             <collision>
                 <geometry>
-                    <mesh filename="package://nano/meshes/wheel.dae" scale="0.6 0.6 0.6" />
+                    <mesh filename="package://aio_robot/meshes/wheel.dae" scale="0.6 0.6 0.6" />
                 </geometry>
                 <origin rpy="${rot} 0 0" xyz="0 0 0.0" />

Commit message: adding camera link to robot model

File: urdf/model.urdf.xacro (robot description, xacro)
@@ -66,3 +66,9 @@
         <child link="laser" />
     </joint>
+    <link name="cam0" pose="0.15011 0 0 0 0 0"/>
+    <joint name="camera_joint" type="fixed">
+        <origin xyz="0.0 0.00 0.0" rpy="0 0 0" />
+        <parent link="base_link" />
+        <child link="cam0" />
+    </joint>
 </robot>

Commit message: change in link name

File: urdf/model.urdf.xacro (robot description, xacro)
@@ -66,5 +66,5 @@
         <child link="laser" />
     </joint>
-    <link name="cam0" pose="0.15011 0 0 0 0 0"/>
+    <link name="cam0_link" pose="0.15011 0 0 0 0 0"/>
     <joint name="camera_joint" type="fixed">
         <origin xyz="0.0 0.00 0.0" rpy="0 0 0" />

Commit message: change in robot model

File: urdf/model.urdf.xacro (robot description, xacro)
@@ -70,5 +70,5 @@
         <origin xyz="0.0 0.00 0.0" rpy="0 0 0" />
         <parent link="base_link" />
-        <child link="cam0" />
+        <child link="cam0_link" />
     </joint>
 </robot>

Commit message: adjust the urdf camera link, joint, geometry

File: urdf/model.urdf.xacro (robot description, xacro)
@@ -66,7 +66,14 @@
         <child link="laser" />
     </joint>
-    <link name="cam0_link" pose="0.15011 0 0 0 0 0"/>
+    <link name="cam0_link" pose="0.0 0 0 0 0 0">
+    <visual>
+        <origin xyz="0 0 0" rpy="0 0 0" />
+        <geometry>
+            <sphere  radius="0.01" />
+        </geometry>
+    </visual>
+    </link>
     <joint name="camera_joint" type="fixed">
-        <origin xyz="0.0 0.00 0.0" rpy="0 0 0" />
+        <origin xyz="0.145 0.00 0.0" rpy="0 0 0" />
         <parent link="base_link" />
         <child link="cam0_link" />
